File: kicad/display.kicad_sch (KiCad schematic)
At the start: 17 parts, among them J5 Conn_01x18, Q1 Si1308EDL

Commit message: moving things around
Parts:
- J4: renamed from J5; footprint (none) -> Connector_FFC-FPC:Amphenol_F32Q-1A7x1-11018_1x18-1MP_P0.5mm_Horizontal
- L1: footprint (none) -> Inductor_SMD:L_0805_2012Metric_Pad1.05x1.20mm_HandSolder
- renumbered C23 to C19, C27 to C20, C26 to C21, C25 to C22, C24 to C23, C21 to C24, C20 to C25, C22 to C26, C19 to C27, D65 to D67, D64 to D68
Changed lines of the file:
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@@
 		(on_board yes)
 		(dnp no)
-		(property "Reference" "C24"
+		(property "Reference" "C23"
 			(at 201.93 76.2 90)
 			(effects
@@
 			(project "keyboard"
 				(path "/6dbb65f4-5576-4e18-9627-83014d84ecc4/e7e875cf-efe4-43d8-ad3f-d0327ce74593"
-					(reference "C24")
+					(reference "C23")
 					(unit 1)
 				)
@@
 		(dnp no)
 		(fields_autoplaced yes)
-		(property "Reference" "J5"
+		(property "Reference" "J4"
 			(at 236.22 52.0699 0)
 			(effects
@@
 			)
 		)
-		(property "Footprint" ""
+		(property "Footprint" "Connector_FFC-FPC:Amphenol_F32Q-1A7x1-11018_1x18-1MP_P0.5mm_Horizontal"
 			(at 233.68 52.07 0)
 			(effects
@@
 			(project ""
 				(path "/6dbb65f4-5576-4e18-9627-83014d84ecc4/e7e875cf-efe4-43d8-ad3f-d0327ce74593"
-					(reference "J5")
+					(reference "J4")
 					(unit 1)
 				)
@@
 		(on_board yes)
 		(dnp no)
-		(property "Reference" "#PWR041"
+		(property "Reference" "#PWR037"
 			(at 222.25 57.15 0)
 			(effects
@@
 			(project "keyboard"
 				(path "/6dbb65f4-5576-4e18-9627-83014d84ecc4/e7e875cf-efe4-43d8-ad3f-d0327ce74593"
-					(reference "#PWR041")
+					(reference "#PWR037")
 					(unit 1)
 				)
@@
 		(on_board yes)
 		(dnp no)
-		(property "Reference" "C23"
+		(property "Reference" "C19"
 			(at 189.611 44.5516 0)
 			(effects
@@
 			(project "keyboard"
 				(path "/6dbb65f4-5576-4e18-9627-83014d84ecc4/e7e875cf-efe4-43d8-ad3f-d0327ce74593"
-					(reference "C23")
+					(reference "C19")
 					(unit 1)
 				)
@@
 		(dnp no)
 		(fields_autoplaced yes)
-		(property "Reference" "D65"
+		(property "Reference" "D67"
 			(at 100.6475 88.9 0)
 			(effects
@@
 			(project "keyboard"
 				(path "/6dbb65f4-5576-4e18-9627-83014d84ecc4/e7e875cf-efe4-43d8-ad3f-d0327ce74593"
-					(reference "D65")
+					(reference "D67")
 					(unit 1)
 				)
@@
 		(on_board yes)
 		(dnp no)
-		(property "Reference" "#PWR043"
+		(property "Reference" "#PWR038"
 			(at 186.69 90.17 0)
 			(effects
@@
 			(project "keyboard"
 				(path "/6dbb65f4-5576-4e18-9627-83014d84ecc4/e7e875cf-efe4-43d8-ad3f-d0327ce74593"
-					(reference "#PWR043")
+					(reference "#PWR038")
 					(unit 1)
 				)
@@
 		(on_board yes)
 		(dnp no)
-		(property "Reference" "#PWR039"
+		(property "Reference" "#PWR040"
 			(at 110.49 101.6 0)
 			(effects
@@
 			(project "keyboard"
 				(path "/6dbb65f4-5576-4e18-9627-83014d84ecc4/e7e875cf-efe4-43d8-ad3f-d0327ce74593"
-					(reference "#PWR039")
+					(reference "#PWR040")
 					(unit 1)
 				)
@@
 		(on_board yes)
 		(dnp no)
-		(property "Reference" "#PWR040"
+		(property "Reference" "#PWR042"
 			(at 110.49 125.73 0)
 			(effects
@@
 			(project "keyboard"
 				(path "/6dbb65f4-5576-4e18-9627-83014d84ecc4/e7e875cf-efe4-43d8-ad3f-d0327ce74593"
-					(reference "#PWR040")
+					(reference "#PWR042")
 					(unit 1)
 				)
@@
 		(on_board yes)
 		(dnp no)
-		(property "Reference" "C25"
+		(property "Reference" "C22"
 			(at 201.93 67.31 90)
 			(effects
@@
 			(project "keyboard"
 				(path "/6dbb65f4-5576-4e18-9627-83014d84ecc4/e7e875cf-efe4-43d8-ad3f-d0327ce74593"
-					(reference "C25")
+					(reference "C22")
 					(unit 1)
 				)
@@
 		(on_board yes)
 		(dnp no)
-		(property "Reference" "C19"
+		(property "Reference" "C27"
 			(at 61.341 113.1316 0)
 			(effects
@@
 			(project "keyboard"
 				(path "/6dbb65f4-5576-4e18-9627-83014d84ecc4/e7e875cf-efe4-43d8-ad3f-d0327ce74593"
-					(reference "C19")
+					(reference "C27")
 					(unit 1)
 				)
@@
 		(on_board yes)
 		(dnp no)
-		(property "Reference" "C22"
+		(property "Reference" "C26"
 			(at 113.411 110.5916 0)
 			(effects
@@
 			(project "keyboard"
 				(path "/6dbb65f4-5576-4e18-9627-83014d84ecc4/e7e875cf-efe4-43d8-ad3f-d0327ce74593"
-					(reference "C22")
+					(reference "C26")
 					(unit 1)
 				)
@@
 		(on_board yes)
 		(dnp no)
-		(property "Reference" "#PWR047"
+		(property "Reference" "#PWR044"
 			(at 88.9 152.4 0)
 			(effects
@@
 			(project "keyboard"
 				(path "/6dbb65f4-5576-4e18-9627-83014d84ecc4/e7e875cf-efe4-43d8-ad3f-d0327ce74593"
-					(reference "#PWR047")
+					(reference "#PWR044")
 					(unit 1)
 				)
@@
 		(on_board yes)
 		(dnp no)
-		(property "Reference" "C26"
+		(property "Reference" "C21"
 			(at 201.93 63.5 90)
 			(effects
@@
 			(project "keyboard"
 				(path "/6dbb65f4-5576-4e18-9627-83014d84ecc4/e7e875cf-efe4-43d8-ad3f-d0327ce74593"
-					(reference "C26")
+					(reference "C21")
 					(unit 1)
 				)
@@
 		(on_board yes)
 		(dnp no)
-		(property "Reference" "#PWR037"
+		(property "Reference" "#PWR043"
 			(at 58.42 129.54 0)
 			(effects
@@
 			(project "keyboard"
 				(path "/6dbb65f4-5576-4e18-9627-83014d84ecc4/e7e875cf-efe4-43d8-ad3f-d0327ce74593"
-					(reference "#PWR037")
+					(reference "#PWR043")
 					(unit 1)
 				)
@@
 		(on_board yes)
 		(dnp no)
-		(property "Reference" "#PWR042"
+		(property "Reference" "#PWR035"
 			(at 186.69 55.88 0)
 			(effects
@@
 			(project "keyboard"
 				(path "/6dbb65f4-5576-4e18-9627-83014d84ecc4/e7e875cf-efe4-43d8-ad3f-d0327ce74593"
-					(reference "#PWR042")
+					(reference "#PWR035")
 					(unit 1)
 				)
@@
 		(dnp no)
 		(fields_autoplaced yes)
-		(property "Reference" "#PWR035"
+		(property "Reference" "#PWR036"
 			(at 232.41 54.61 0)
 			(effects
@@
 			(project "keyboard"
 				(path "/6dbb65f4-5576-4e18-9627-83014d84ecc4/e7e875cf-efe4-43d8-ad3f-d0327ce74593"
-					(reference "#PWR035")
+					(reference "#PWR036")
 					(unit 1)
 				)
@@
 		(dnp no)
 		(fields_autoplaced yes)
-		(property "Reference" "#PWR036"
+		(property "Reference" "#PWR041"
 			(at 58.42 104.14 0)
 			(effects
@@
 			(project "keyboard"
 				(path "/6dbb65f4-5576-4e18-9627-83014d84ecc4/e7e875cf-efe4-43d8-ad3f-d0327ce74593"
-					(reference "#PWR036")
+					(reference "#PWR041")
 					(unit 1)
 				)
@@
 		(on_board yes)
 		(dnp no)
-		(property "Reference" "#PWR038"
+		(property "Reference" "#PWR039"
 			(at 119.38 99.06 0)
 			(effects
@@
 			(project "keyboard"
 				(path "/6dbb65f4-5576-4e18-9627-83014d84ecc4/e7e875cf-efe4-43d8-ad3f-d0327ce74593"
-					(reference "#PWR038")
+					(reference "#PWR039")
 					(unit 1)
 				)
@@
 		(on_board yes)
 		(dnp no)
-		(property "Reference" "C27"
+		(property "Reference" "C20"
 			(at 201.93 59.69 90)
 			(effects
@@
 			(project "keyboard"
 				(path "/6dbb65f4-5576-4e18-9627-83014d84ecc4/e7e875cf-efe4-43d8-ad3f-d0327ce74593"
-					(reference "C27")
+					(reference "C20")
 					(unit 1)
 				)
@@
 		(dnp no)
 		(fields_autoplaced yes)
-		(property "Reference" "D64"
+		(property "Reference" "D68"
 			(at 100.6475 101.6 0)
 			(effects
@@
 			(project ""
 				(path "/6dbb65f4-5576-4e18-9627-83014d84ecc4/e7e875cf-efe4-43d8-ad3f-d0327ce74593"
-					(reference "D64")
+					(reference "D68")
 					(unit 1)
 				)
@@
 			)
 		)
-		(property "Footprint" ""
+		(property "Footprint" "Inductor_SMD:L_0805_2012Metric_Pad1.05x1.20mm_HandSolder"
 			(at 71.12 107.95 0)
 			(effects
@@
 		(on_board yes)
 		(dnp no)
-		(property "Reference" "C21"
+		(property "Reference" "C24"
 			(at 122.301 87.7316 0)
 			(effects
@@
 			(project "keyboard"
 				(path "/6dbb65f4-5576-4e18-9627-83014d84ecc4/e7e875cf-efe4-43d8-ad3f-d0327ce74593"
-					(reference "C21")
+					(reference "C24")
 					(unit 1)
 				)
@@
 		(on_board yes)
 		(dnp no)
-		(property "Reference" "C20"
+		(property "Reference" "C25"
 			(at 91.821 100.4316 0)
 			(effects
@@
 			(project "keyboard"
 				(path "/6dbb65f4-5576-4e18-9627-83014d84ecc4/e7e875cf-efe4-43d8-ad3f-d0327ce74593"
-					(reference "C20")
-					(unit 1)
-				)
+					(reference "C25")
+					(unit 1)
+				)
