File: kicad/flash.kicad_sch (KiCad schematic)
At the start: 5 parts, among them SW1 SW_DIP_x01, U2 W25Q128JVS

Commit message: moving things around
Parts:
- U2: footprint Package_SO:SOIC-8_5.23x5.23mm_P1.27mm -> Package_SO:SOIC-8_5.3x5.3mm_P1.27mm
- renumbered R3 to R4, R4 to R5
Changed lines of the file:
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@@
 		(on_board yes)
 		(dnp no)
-		(property "Reference" "R3"
+		(property "Reference" "R4"
 			(at 112.268 82.6516 0)
 			(effects
@@
 			(project "keyboard"
 				(path "/6dbb65f4-5576-4e18-9627-83014d84ecc4/7adace9b-063e-4b7c-921f-8b942603049c"
-					(reference "R3")
+					(reference "R4")
 					(unit 1)
 				)
@@
 		(dnp no)
 		(fields_autoplaced yes)
-		(property "Reference" "#PWR012"
+		(property "Reference" "#PWR013"
 			(at 63.5 105.41 0)
 			(effects
@@
 			(project ""
 				(path "/6dbb65f4-5576-4e18-9627-83014d84ecc4/7adace9b-063e-4b7c-921f-8b942603049c"
-					(reference "#PWR012")
+					(reference "#PWR013")
 					(unit 1)
 				)
@@
 		(on_board yes)
 		(dnp no)
-		(property "Reference" "R4"
+		(property "Reference" "R5"
 			(at 95.25 93.8022 90)
 			(effects
@@
 			(project "keyboard"
 				(path "/6dbb65f4-5576-4e18-9627-83014d84ecc4/7adace9b-063e-4b7c-921f-8b942603049c"
-					(reference "R4")
+					(reference "R5")
 					(unit 1)
 				)
@@
 		(on_board yes)
 		(dnp no)
-		(property "Reference" "#PWR013"
+		(property "Reference" "#PWR014"
 			(at 144.78 125.73 0)
 			(effects
@@
 			(project "keyboard"
 				(path "/6dbb65f4-5576-4e18-9627-83014d84ecc4/7adace9b-063e-4b7c-921f-8b942603049c"
-					(reference "#PWR013")
+					(reference "#PWR014")
 					(unit 1)
 				)
@@
 			)
 		)
-		(property "Footprint" "Package_SO:SOIC-8_5.23x5.23mm_P1.27mm"
+		(property "Footprint" "Package_SO:SOIC-8_5.3x5.3mm_P1.27mm"
 			(at 144.78 106.68 0)
 			(effects
@@
 		(on_board yes)
 		(dnp no)
-		(property "Reference" "#PWR010"
+		(property "Reference" "#PWR011"
 			(at 144.78 77.47 0)
 			(effects
@@
 			(project "keyboard"
 				(path "/6dbb65f4-5576-4e18-9627-83014d84ecc4/7adace9b-063e-4b7c-921f-8b942603049c"
-					(reference "#PWR010")
+					(reference "#PWR011")
 					(unit 1)
 				)
@@
 		(on_board yes)
 		(dnp no)
-		(property "Reference" "#PWR011"
+		(property "Reference" "#PWR012"
 			(at 151.13 91.44 0)
 			(effects
@@
 			(project "keyboard"
 				(path "/6dbb65f4-5576-4e18-9627-83014d84ecc4/7adace9b-063e-4b7c-921f-8b942603049c"
-					(reference "#PWR011")
-					(unit 1)
-				)
+					(reference "#PWR012")
+					(unit 1)
+				)
