File: kicad/oscillator.kicad_sch (KiCad schematic)
At the start: 4 parts, among them Y1 ABM8-272-T3

Commit message: moving things around
Parts:
- renumbered R5 to R6
Changed lines of the file:
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@@
 		(on_board yes)
 		(dnp no)
-		(property "Reference" "#PWR014"
+		(property "Reference" "#PWR015"
 			(at 107.95 120.65 0)
 			(effects
@@
 			(project "keyboard"
 				(path "/6dbb65f4-5576-4e18-9627-83014d84ecc4/31815c76-57e3-46f4-a3e7-b464abc06b3f"
-					(reference "#PWR014")
+					(reference "#PWR015")
 					(unit 1)
 				)
@@
 		(on_board yes)
 		(dnp no)
-		(property "Reference" "#PWR016"
+		(property "Reference" "#PWR017"
 			(at 92.71 128.27 0)
 			(effects
@@
 			(project "keyboard"
 				(path "/6dbb65f4-5576-4e18-9627-83014d84ecc4/31815c76-57e3-46f4-a3e7-b464abc06b3f"
-					(reference "#PWR016")
+					(reference "#PWR017")
 					(unit 1)
 				)
@@
 		(on_board yes)
 		(dnp no)
-		(property "Reference" "#PWR015"
+		(property "Reference" "#PWR016"
 			(at 120.65 120.65 0)
 			(effects
@@
 			(project "keyboard"
 				(path "/6dbb65f4-5576-4e18-9627-83014d84ecc4/31815c76-57e3-46f4-a3e7-b464abc06b3f"
-					(reference "#PWR015")
+					(reference "#PWR016")
 					(unit 1)
 				)
@@
 		(on_board yes)
 		(dnp no)
-		(property "Reference" "R5"
+		(property "Reference" "R6"
 			(at 132.08 114.1222 90)
 			(effects
@@
 			(project "keyboard"
 				(path "/6dbb65f4-5576-4e18-9627-83014d84ecc4/31815c76-57e3-46f4-a3e7-b464abc06b3f"
-					(reference "R5")
-					(unit 1)
-				)
+					(reference "R6")
+					(unit 1)
+				)
