File: kicad/switchmat.kicad_sch (KiCad schematic)
At the start: 136 parts, among them SW10 SW_Push, SW11 SW_Push, SW12 SW_Push, SW13 SW_Push, SW14 SW_Push, SW15 SW_Push, SW16 SW_Push, SW17 SW_Push, SW18 SW_Push, SW19 SW_Push, SW20 SW_Push, SW21 SW_Push, SW22 SW_Push, SW23 SW_Push, SW24 SW_Push, SW25 SW_Push, SW26 SW_Push, SW27 SW_Push, SW28 SW_Push, SW29 SW_Push, SW3 SW_Push, SW30 SW_Push, SW31 SW_Push, SW32 SW_Push, SW33 SW_Push, SW34 SW_Push, SW35 SW_Push, SW36 SW_Push, SW37 SW_Push, SW38 SW_Push, SW39 SW_Push, SW4 SW_Push, SW40 SW_Push, SW41 SW_Push, SW42 SW_Push, SW43 SW_Push, SW44 SW_Push, SW45 SW_Push, SW46 SW_Push, SW47 SW_Push, SW48 SW_Push, SW49 SW_Push, SW5 SW_Push, SW50 SW_Push, SW51 SW_Push, SW52 SW_Push, SW53 SW_Push, SW54 SW_Push, SW55 SW_Push, SW56 SW_Push, SW57 SW_Push, SW58 SW_Push, SW59 SW_Push, SW6 SW_Push, SW60 SW_Push, SW61 SW_Push, SW62 SW_Push, SW63 SW_Push, SW64 SW_Push, SW65 SW_Push, SW66 SW_Push, SW67 SW_Push, SW68 SW_Push, SW69 SW_Push, SW7 SW_Push, SW70 SW_Push, SW8 SW_Push, SW9 SW_Push

Commit message: actual attempt at source controlling kicad project
Parts:
- removed D14, D15, D29, D30, D44, D57, D60, D65, D66: 1N4148WT, Diode_SMD:D_SOD-523, symbol Diode:1N4148WT
- removed SW16, SW17, SW31, SW32, SW46, SW59, SW69, SW70: SW_Push, Button_Switch_Keyboard:SW_Cherry_MX_1.00u_PCB, symbol Switch:SW_Push
- removed SW62: SW_Push, Button_Switch_Keyboard:SW_Cherry_MX_1.25u_PCB, symbol Switch:SW_Push
- added D18, D36, D45, D59, D68: 1N4148WT, Diode_SMD:D_SOD-523, symbol Diode:1N4148WT
- added SW20, SW67: SW_Push, Button_Switch_Keyboard:SW_Cherry_MX_1.25u_PCB, symbol Switch:SW_Push
- added SW38: SW_Push, Button_Switch_Keyboard:SW_Cherry_MX_6.25u_PCB, symbol Switch:SW_Push
- added SW47: SW_Push, Button_Switch_Keyboard:SW_Cherry_MX_1.00u_PCB, symbol Switch:SW_Push
- added SW61: SW_Push, PCM_Switch_Keyboard_Cherry_MX:SW_Cherry_MX_Plate_1.75u, symbol Switch:SW_Push
- SW60: footprint Button_Switch_Keyboard:SW_Cherry_MX_1.00u_PCB -> PCM_Switch_Keyboard_Cherry_MX:SW_Cherry_MX_Plate_1.75u
- renumbered D18 to D10, D33 to D11, D46 to D12, D61 to D13, D4 to D14, D19 to D15, D34 to D16, D47 to D17, D5 to D19, D16 to D2, D35 to D21, D48 to D22, D6 to D23, D21 to D24, D36 to D25, D49 to D26, D62 to D27, D7 to D28, D22 to D29, D31 to D3, D37 to D30, D50 to D31, D8 to D32, D23 to D33, D38 to D34, D51 to D35, D9 to D37, D24 to D38, D45 to D4, D52 to D40, D10 to D41, D25 to D42, D40 to D43, D53 to D44, D11 to D46, D26 to D47, D41 to D48, D54 to D49, D59 to D5, D63 to D50, D12 to D51, D27 to D52, D42 to D53, D55 to D54, D69 to D55, D13 to D56, D28 to D57, D2 to D6, D70 to D60, D43 to D61, D56 to D62, D64 to D63, D17 to D7, D32 to D8, D3 to D9, SW34 to SW10, SW5 to SW11, SW20 to SW12, SW35 to SW13, SW48 to SW14, SW63 to SW15, SW6 to SW16, SW21 to SW17, SW36 to SW18, SW49 to SW19, SW7 to SW21, SW37 to SW23, SW50 to SW24, SW8 to SW25, SW23 to SW26, SW38 to SW27, SW51 to SW28, SW64 to SW29, SW9 to SW30, SW24 to SW31, SW39 to SW32, SW52 to SW33, SW10 to SW34, SW25 to SW35, SW40 to SW36, SW53 to SW37, SW11 to SW39, SW18 to SW4, SW26 to SW40, SW54 to SW42, SW12 to SW43, SW27 to SW44, SW42 to SW45, SW55 to SW46, SW13 to SW48, SW28 to SW49, SW33 to SW5, SW43 to SW50, SW56 to SW51, SW65 to SW52, SW14 to SW53, SW29 to SW54, SW44 to SW55, SW57 to SW56, SW66 to SW57, SW15 to SW58, SW30 to SW59, SW47 to SW6, SW67 to SW62, SW45 to SW63, SW58 to SW64, SW68 to SW65, SW61 to SW7, SW4 to SW8, SW19 to SW9
Connections:
- net Col15 is gone; now on net Col12: D58.1 (K)
- net Col1: now also D68.1 (K)
- net Col12: now also D59.1 (K)
- net Col4: now also D18.1 (K)
- net Col5: now also D27.1 (K)
- net Col6: no longer D27.1 (K)
- net Col7: now also D36.1 (K)
- net Col9: now also D45.1 (K)
- net Row1: now also SW63.1
- net Row2: now also SW60.1; no longer SW63.1
- net Row3: now also SW61.1; no longer SW60.1
- net Row4: now also SW20.1, SW38.1, SW47.1, SW67.1
- new net: D36.2 (A), SW38.2
- new net: D59.2 (A), SW61.2
- new net: D18.2 (A), SW20.2
- new net: D68.2 (A), SW67.2
- new net: D45.2 (A), SW47.2
Other:
- moved on the sheet: D27, D61, SW29, SW63

Commit message: moving things around
Parts:
- D10: renamed from D37; footprint Diode_SMD:D_SOD-523 -> Diode_SMD:D_SOD-323_HandSoldering
- D11: renamed from D41; footprint Diode_SMD:D_SOD-523 -> Diode_SMD:D_SOD-323_HandSoldering
- D12: renamed from D46; footprint Diode_SMD:D_SOD-523 -> Diode_SMD:D_SOD-323_HandSoldering
- D13: renamed from D51; footprint Diode_SMD:D_SOD-523 -> Diode_SMD:D_SOD-323_HandSoldering
- D14: renamed from D56; footprint Diode_SMD:D_SOD-523 -> Diode_SMD:D_SOD-323_HandSoldering
- D15: renamed from D2; footprint Diode_SMD:D_SOD-523 -> Diode_SMD:D_SOD-323_HandSoldering
- D16: renamed from D7; footprint Diode_SMD:D_SOD-523 -> Diode_SMD:D_SOD-323_HandSoldering
- D17: renamed from D10; footprint Diode_SMD:D_SOD-523 -> Diode_SMD:D_SOD-323_HandSoldering
- D18: renamed from D15; footprint Diode_SMD:D_SOD-523 -> Diode_SMD:D_SOD-323_HandSoldering
- D19: renamed from D20; footprint Diode_SMD:D_SOD-523 -> Diode_SMD:D_SOD-323_HandSoldering
- D2: renamed from D1; footprint Diode_SMD:D_SOD-523 -> Diode_SMD:D_SOD-323_HandSoldering
- D20: renamed from D24; footprint Diode_SMD:D_SOD-523 -> Diode_SMD:D_SOD-323_HandSoldering
- D21: renamed from D29; footprint Diode_SMD:D_SOD-523 -> Diode_SMD:D_SOD-323_HandSoldering
- D22: renamed from D33; footprint Diode_SMD:D_SOD-523 -> Diode_SMD:D_SOD-323_HandSoldering
- D23: renamed from D38; footprint Diode_SMD:D_SOD-523 -> Diode_SMD:D_SOD-323_HandSoldering
- D24: renamed from D42; footprint Diode_SMD:D_SOD-523 -> Diode_SMD:D_SOD-323_HandSoldering
- D25: renamed from D47; footprint Diode_SMD:D_SOD-523 -> Diode_SMD:D_SOD-323_HandSoldering
- D26: renamed from D52; footprint Diode_SMD:D_SOD-523 -> Diode_SMD:D_SOD-323_HandSoldering
- D27: renamed from D57; footprint Diode_SMD:D_SOD-523 -> Diode_SMD:D_SOD-323_HandSoldering
- D28: renamed from D61; footprint Diode_SMD:D_SOD-523 -> Diode_SMD:D_SOD-323_HandSoldering
- D29: renamed from D3; footprint Diode_SMD:D_SOD-523 -> Diode_SMD:D_SOD-323_HandSoldering
- D3: renamed from D6; footprint Diode_SMD:D_SOD-523 -> Diode_SMD:D_SOD-323_HandSoldering
- D30: renamed from D8; footprint Diode_SMD:D_SOD-523 -> Diode_SMD:D_SOD-323_HandSoldering
- D31: renamed from D11; footprint Diode_SMD:D_SOD-523 -> Diode_SMD:D_SOD-323_HandSoldering
- D32: renamed from D16; footprint Diode_SMD:D_SOD-523 -> Diode_SMD:D_SOD-323_HandSoldering
- D33: renamed from D21; footprint Diode_SMD:D_SOD-523 -> Diode_SMD:D_SOD-323_HandSoldering
- D34: renamed from D25; footprint Diode_SMD:D_SOD-523 -> Diode_SMD:D_SOD-323_HandSoldering
- D35: renamed from D30; footprint Diode_SMD:D_SOD-523 -> Diode_SMD:D_SOD-323_HandSoldering
- D36: renamed from D34; footprint Diode_SMD:D_SOD-523 -> Diode_SMD:D_SOD-323_HandSoldering
- D37: renamed from D39; footprint Diode_SMD:D_SOD-523 -> Diode_SMD:D_SOD-323_HandSoldering
- D38: renamed from D43; footprint Diode_SMD:D_SOD-523 -> Diode_SMD:D_SOD-323_HandSoldering
- D39: renamed from D48; footprint Diode_SMD:D_SOD-523 -> Diode_SMD:D_SOD-323_HandSoldering
- D4: renamed from D9; footprint Diode_SMD:D_SOD-523 -> Diode_SMD:D_SOD-323_HandSoldering
- D40: renamed from D53; footprint Diode_SMD:D_SOD-523 -> Diode_SMD:D_SOD-323_HandSoldering
- D41: renamed from D58; footprint Diode_SMD:D_SOD-523 -> Diode_SMD:D_SOD-323_HandSoldering
- D42: renamed from D4; footprint Diode_SMD:D_SOD-523 -> Diode_SMD:D_SOD-323_HandSoldering
- D43: renamed from D12; footprint Diode_SMD:D_SOD-523 -> Diode_SMD:D_SOD-323_HandSoldering
- D44: renamed from D17; footprint Diode_SMD:D_SOD-523 -> Diode_SMD:D_SOD-323_HandSoldering
- D45: renamed from D22; footprint Diode_SMD:D_SOD-523 -> Diode_SMD:D_SOD-323_HandSoldering
- D46: renamed from D26; footprint Diode_SMD:D_SOD-523 -> Diode_SMD:D_SOD-323_HandSoldering
- D47: renamed from D31; footprint Diode_SMD:D_SOD-523 -> Diode_SMD:D_SOD-323_HandSoldering
- D48: renamed from D35; footprint Diode_SMD:D_SOD-523 -> Diode_SMD:D_SOD-323_HandSoldering
- D49: renamed from D40; footprint Diode_SMD:D_SOD-523 -> Diode_SMD:D_SOD-323_HandSoldering
- D5: renamed from D14; footprint Diode_SMD:D_SOD-523 -> Diode_SMD:D_SOD-323_HandSoldering
- D50: renamed from D44; footprint Diode_SMD:D_SOD-523 -> Diode_SMD:D_SOD-323_HandSoldering
- D51: renamed from D49; footprint Diode_SMD:D_SOD-523 -> Diode_SMD:D_SOD-323_HandSoldering
- D52: renamed from D54; footprint Diode_SMD:D_SOD-523 -> Diode_SMD:D_SOD-323_HandSoldering
- D53: renamed from D59; footprint Diode_SMD:D_SOD-523 -> Diode_SMD:D_SOD-323_HandSoldering
- D54: renamed from D62; footprint Diode_SMD:D_SOD-523 -> Diode_SMD:D_SOD-323_HandSoldering
- D55: renamed from D5; footprint Diode_SMD:D_SOD-523 -> Diode_SMD:D_SOD-323_HandSoldering
- D57: renamed from D13; footprint Diode_SMD:D_SOD-523 -> Diode_SMD:D_SOD-323_HandSoldering
- D58: renamed from D18; footprint Diode_SMD:D_SOD-523 -> Diode_SMD:D_SOD-323_HandSoldering
- D59: renamed from D27; footprint Diode_SMD:D_SOD-523 -> Diode_SMD:D_SOD-323_HandSoldering
- D6: renamed from D19; footprint Diode_SMD:D_SOD-523 -> Diode_SMD:D_SOD-323_HandSoldering
- D60: renamed from D36; footprint Diode_SMD:D_SOD-523 -> Diode_SMD:D_SOD-323_HandSoldering
- D61: renamed from D45; footprint Diode_SMD:D_SOD-523 -> Diode_SMD:D_SOD-323_HandSoldering
- D62: renamed from D50; footprint Diode_SMD:D_SOD-523 -> Diode_SMD:D_SOD-323_HandSoldering
- D63: renamed from D55; footprint Diode_SMD:D_SOD-523 -> Diode_SMD:D_SOD-323_HandSoldering
- D64: renamed from D60; footprint Diode_SMD:D_SOD-523 -> Diode_SMD:D_SOD-323_HandSoldering
- D65: renamed from D63; footprint Diode_SMD:D_SOD-523 -> Diode_SMD:D_SOD-323_HandSoldering
- D7: renamed from D23; footprint Diode_SMD:D_SOD-523 -> Diode_SMD:D_SOD-323_HandSoldering
- D8: renamed from D28; footprint Diode_SMD:D_SOD-523 -> Diode_SMD:D_SOD-323_HandSoldering
- D9: renamed from D32; footprint Diode_SMD:D_SOD-523 -> Diode_SMD:D_SOD-323_HandSoldering
- SW19: renamed from SW4; footprint Button_Switch_Keyboard:SW_Cherry_MX_1.50u_PCB -> Button_Switch_Keyboard:SW_Cherry_MX_1.00u_PCB
- SW32: renamed from SW63; footprint Button_Switch_Keyboard:SW_Cherry_MX_2.25u_PCB -> Button_Switch_Keyboard:SW_Cherry_MX_1.00u_PCB
- SW33: renamed from SW5; footprint PCM_Switch_Keyboard_Cherry_MX:SW_Cherry_MX_Plate_1.75u -> Button_Switch_Keyboard:SW_Cherry_MX_1.25u_PCB
- SW45: renamed from SW60; footprint PCM_Switch_Keyboard_Cherry_MX:SW_Cherry_MX_Plate_1.75u -> Button_Switch_Keyboard:SW_Cherry_MX_1.75u_PCB
- SW46: renamed from SW6; footprint Button_Switch_Keyboard:SW_Cherry_MX_2.25u_PCB -> Button_Switch_Keyboard:SW_Cherry_MX_1.75u_PCB
- SW57: renamed from SW61; footprint PCM_Switch_Keyboard_Cherry_MX:SW_Cherry_MX_Plate_1.75u -> Button_Switch_Keyboard:SW_Cherry_MX_1.25u_PCB
- SW58: renamed from SW64; footprint PCM_Switch_Keyboard_Cherry_MX:SW_Cherry_MX_Plate_1.75u -> Button_Switch_Keyboard:SW_Cherry_MX_1.00u_PCB
- SW6: renamed from SW3; footprint Button_Switch_Keyboard:SW_Cherry_MX_1.00u_PCB -> Button_Switch_Keyboard:SW_Cherry_MX_1.25u_PCB
- SW60: renamed from SW67; footprint Button_Switch_Keyboard:SW_Cherry_MX_1.25u_PCB -> Button_Switch_Keyboard:SW_Cherry_MX_1.00u_PCB
- SW63: renamed from SW29; footprint Button_Switch_Keyboard:SW_Cherry_MX_6.25u_PCB -> Button_Switch_Keyboard:SW_Cherry_MX_1.75u_PCB
- SW64: renamed from SW38; footprint Button_Switch_Keyboard:SW_Cherry_MX_6.25u_PCB -> Button_Switch_Keyboard:SW_Cherry_MX_2.25u_PCB
- SW65: renamed from SW47; footprint Button_Switch_Keyboard:SW_Cherry_MX_1.00u_PCB -> Button_Switch_Keyboard:SW_Cherry_MX_1.25u_PCB
- renumbered D68 to D56, SW21 to SW10, SW25 to SW11, SW30 to SW12, SW34 to SW13, SW39 to SW14, SW43 to SW15, SW48 to SW16, SW53 to SW17, SW58 to SW18, SW9 to SW20, SW12 to SW21, SW17 to SW22, SW22 to SW23, SW26 to SW24, SW31 to SW25, SW35 to SW26, SW40 to SW27, SW44 to SW28, SW49 to SW29, SW54 to SW30, SW59 to SW31, SW10 to SW34, SW13 to SW35, SW18 to SW36, SW23 to SW37, SW27 to SW38, SW32 to SW39, SW36 to SW40, SW45 to SW42, SW50 to SW43, SW55 to SW44, SW14 to SW47, SW19 to SW48, SW24 to SW49, SW28 to SW50, SW33 to SW51, SW37 to SW52, SW42 to SW53, SW46 to SW54, SW51 to SW55, SW7 to SW59, SW15 to SW61, SW20 to SW62, SW52 to SW66, SW57 to SW67, SW62 to SW68, SW65 to SW69, SW8 to SW7, SW11 to SW8, SW16 to SW9
